File: KiCad Projects/Uno/Arduino UNO R4 WiFi/Arduino UNO R4 WiFi.kicad_pcb (KiCad board)
At the start: 4 copper layers, 68.6 x 53.3 mm, 262 parts, among them J1 USB_C_Receptacle_USB2.0_16P, J10 M20-9990345, J2 SM04B-SRSS-TB(LF)(SN), J3 M20-9980345, J4 PPTC081LFBN-RC, J5 PJ-102AH, J6 M20-9980345, J7 PPTC061LFBN-RC, J8 PPTC101LFBN-RC, J9 PPTC081LFBN-RC, M1 ESP32-S3-MINI-1-N8, Q1 2N7002KT1G, Q2 2N7002KT1G, Q3 2N7002KT1G, U1 R7FA4M1AB3CFM#AA0, U2 TS5A3159ADCK, U3 ISL854102FRZ-T, U4 TXB0108DQSR, U5 AP7361C-33E, U6 TS5A3159ADCK

Commit message: Replace files
Parts:
- moved R40 2.16 mm to (141.5, 106.4)
- moved C14 1.04 mm to (140.5, 106.4)
- moved R38 0.94 mm to (139.5, 106.4)
- moved R36 0.31 mm to (142.2, 104.1)
- turned C2 to 180 degrees
Routing:
- net GND: track 113.1 -> 358.4 mm, vias 83 -> 107
- net +5V: track 128.0 -> 209.8 mm, vias 23 -> 33
- net RA4_P: track 52.0 -> 48.6 mm
- net P004: track 37.2 -> 39.3 mm
- net Net-(C14-Pad1): track 15.2 -> 17.1 mm, vias 0 -> 2
- net ROW5: track 74.9 -> 74.0 mm, vias 7 -> 6
- net P408: track 59.7 -> 60.5 mm
- net P102_SPI0_RSPCK_GPT2_B_CAN0_RX: track 94.3 -> 93.5 mm
- net P002_AN02_AMPO: track 63.2 -> 62.5 mm
- net P001_AN01_AMP-: track 64.1 -> 63.4 mm
- net P000_AN00_AMP+: track 66.4 -> 65.7 mm
- net P300_SWCLK: track 67.0 -> 67.6 mm
- net P100_AN22_SCL: track 108.2 -> 107.7 mm
- net P213: track 40.4 -> 39.8 mm
- net VREFH0: track 7.42 -> 7.92 mm
- removed copper zone on In2.Cu, net +5V
- removed copper zone on In1.Cu, net GND
- removed copper zone on In2.Cu, net GND
Other:
- copper layers 4 -> 2
- board text added: "GITHUB.COM/SABOGALC GITHUB.COM/DYNAMIBYTE"
- board text removed: "GITHUB.COM/SABOGALC"
